Commit message: Imported upstream version '0.6.3' of 'upstream'

File: schunk_description/urdf/lwa/lwa.urdf.xacro (robot description, xacro)
@@ -5,15 +5,11 @@
   <xacro:macro name="schunk_lwa" params="parent name *origin">
     <!-- joint between base_link and arm_0_link -->
-    <joint name="${name}_0_joint" type="fixed" >
+    <joint name="${name}_base_joint" type="fixed" >
       <insert_block name="origin" />
       <parent link="${parent}" />
-      <child link="${name}_0_link" />
-    </joint>
-    <link name="${name}_0_link">
-      <inertial>
-        <origin xyz="0 0 0" rpy="0 0 0"/>
-        <mass value="1.0"/>
-        <inertia ixx="0.01" ixy="0" ixz="0" iyy="0.01" iyz="0" izz="0.01" />
-      </inertial>
+      <child link="${name}_base_link" />
+    </joint>
+    <link name="${name}_base_link">
+      <xacro:default_inertial/>
       <visual>
         <origin xyz="0 0 0.004" rpy="0 0 0" />
@@ -33,19 +29,14 @@
     <joint name="${name}_1_joint" type="revolute">
       <origin xyz="0 0 -0.250" rpy="0 0 3.1415926"/>
-      <parent link="${name}_0_link"/>
+      <parent link="${name}_base_link"/>
       <child link="${name}_1_link"/>
       <axis xyz="0 0 1"/>
-      <calibration rising="${arm_1_ref}"/>
       <dynamics damping="10" />
-      <limit effort="370" velocity="2.0" lower="-6.25" upper="6.25"/>
-      <safety_controller k_position="20" k_velocity="50" soft_lower_limit="${-6.25 + 0.01}" soft_upper_limit="${6.25 - 0.01}" />
+      <limit effort="370" velocity="2.0" lower="-3.1415" upper="3.1415"/>
+      <!--limit effort="370" velocity="2.0" lower="-6.25" upper="6.25"/-->
+      <!--safety_controller k_position="20" k_velocity="50" soft_lower_limit="${-6.25 + 0.01}" soft_upper_limit="${6.25 - 0.01}" /-->
     </joint>
     <link name="${name}_1_link">
-      <inertial>
-        <origin xyz="0 0 0" rpy="0 0 0" />
-        <!--mass value="5.9907"/-->
-        <mass value="2.0"/>
-        <inertia ixx="0.01" ixy="0" ixz="0" iyy="0.01" iyz="0" izz="0.01" />
-      </inertial>
+      <xacro:default_inertial/>
       <visual>
         <origin xyz="0 0 0" rpy="0 0 0" />
@@ -68,16 +59,10 @@
       <child link="${name}_2_link"/>
       <axis xyz="0 0 1"/>
-      <calibration rising="${arm_2_ref}"/>
       <dynamics damping="10" />
       <limit effort="370" velocity="2.0" lower="-1.97" upper="1.97"/>
-      <safety_controller k_position="20" k_velocity="50" soft_lower_limit="${-1.97 + 0.01}"   soft_upper_limit="${1.97 - 0.01}" />
+      <!--safety_controller k_position="20" k_velocity="50" soft_lower_limit="${-1.97 + 0.01}"   soft_upper_limit="${1.97 - 0.01}" /-->
     </joint>
     <link name="${name}_2_link">
-      <inertial>
-        <origin xyz="0 0 0" rpy="0 0 0"/>
-        <!--mass value="5.734939"/-->
-        <mass value="2.0"/>
-        <inertia ixx="0.03" ixy="0" ixz="0" iyy="0.03" iyz="0" izz="0.03" />
-      </inertial>
+      <xacro:default_inertial/>
       <visual>
         <origin xyz="0 0 0" rpy="0 0 0" />
@@ -100,16 +85,11 @@
       <child link="${name}_3_link"/>
       <axis xyz="0 0 1"/>
-      <calibration rising="${arm_3_ref}"/>
-      <dynamics damping="5" />
-      <limit effort="176" velocity="2.0" lower="-6.25" upper="6.25"/>
-      <safety_controller k_position="20" k_velocity="25" soft_lower_limit="${-6.25 + 0.01}" soft_upper_limit="${6.25 - 0.01}" />
+      <dynamics damping="5" />
+      <limit effort="176" velocity="2.0" lower="-3.1415" upper="3.1415"/>
+      <!--limit effort="176" velocity="2.0" lower="-6.25" upper="6.25"/-->
+      <!--safety_controller k_position="20" k_velocity="25" soft_lower_limit="${-6.25 + 0.01}" soft_upper_limit="${6.25 - 0.01}" /-->
     </joint>
     <link name="${name}_3_link">
-      <inertial>
-        <origin xyz="0 0 0" rpy="0 0 0"/>
-        <!--mass value="4.214668"/-->
-        <mass value="2.0"/>
-        <inertia ixx="0.03" ixy="0" ixz="0" iyy="0.03" iyz="0" izz="0.03" />
-      </inertial>
+      <xacro:default_inertial/>
       <visual>
         <origin xyz="0 0 0" rpy="0 0 0" />
@@ -132,16 +112,10 @@
       <child link="${name}_4_link"/>
       <axis xyz="0 0 1" />
-      <calibration rising="${arm_4_ref}"/>
       <dynamics damping="5" />
       <limit effort="176" velocity="2.0" lower="-1.97" upper="1.97"/>
-      <safety_controller k_position="20" k_velocity="25" soft_lower_limit="${-1.97 + 0.01}" soft_upper_limit="${1.97 - 0.01}" />
+      <!--safety_controller k_position="20" k_velocity="25" soft_lower_limit="${-1.97 + 0.01}" soft_upper_limit="${1.97 - 0.01}" /-->
     </joint>
     <link name="${name}_4_link">
-      <inertial>
-        <origin xyz="0 0 0" rpy="0 0 0"/>
-        <!--mass value="3.669819"/-->
-        <mass value="2.0"/>
-        <inertia ixx="0.03" ixy="0" ixz="0" iyy="0.03" iyz="0" izz="0.03" />
-      </inertial>
+      <xacro:default_inertial/>
       <visual>
         <origin xyz="0 0 0" rpy="0 0 0" />
@@ -164,15 +138,11 @@
       <child link="${name}_5_link"/>
       <axis xyz="0 0 1" />
-      <calibration rising="${arm_5_ref}"/>
-      <dynamics damping="5" />
-      <limit effort="41.6" velocity="2.0" lower="-6.25" upper="6.25" />
-      <safety_controller k_position="20" k_velocity="25" soft_lower_limit="${-6.25 + 0.01}" soft_upper_limit="${6.25 - 0.01}" />
+      <dynamics damping="5" />
+      <limit effort="41.6" velocity="2.0" lower="-3.1415" upper="3.1415" />
+      <!--limit effort="41.6" velocity="2.0" lower="-6.25" upper="6.25" /-->
+      <!--safety_controller k_position="20" k_velocity="25" soft_lower_limit="${-6.25 + 0.01}" soft_upper_limit="${6.25 - 0.01}" /-->
     </joint>
     <link name="${name}_5_link">
-      <inertial>
-        <origin xyz="0 0 0" rpy="0 0 0"/>
-        <mass value="2.313272"/>
-        <inertia ixx="0.03" ixy="0" ixz="0" iyy="0.03" iyz="0" izz="0.03" />
-      </inertial>
+      <xacro:default_inertial/>
       <visual>
         <origin xyz="0 0 0" rpy="0 0 0" />
@@ -195,15 +165,10 @@
       <child link="${name}_6_link"/>
       <axis xyz="0 0 1" />
-      <calibration rising="${arm_6_ref}"/>
       <dynamics damping="5" />
       <limit effort="20.1" velocity="2.0" lower="-1.97" upper="1.97" />
-      <safety_controller k_position="20" k_velocity="25" soft_lower_limit="${-1.97 + 0.01}" soft_upper_limit="${1.97 - 0.01}" />
+      <!--safety_controller k_position="20" k_velocity="25" soft_lower_limit="${-1.97 + 0.01}" soft_upper_limit="${1.97 - 0.01}" /-->
     </joint>
     <link name="${name}_6_link">
-      <inertial>
-        <origin xyz="0 0 0" rpy="0 0 0"/>
-        <mass value="2.057856"/>
-        <inertia ixx="0.01" ixy="0" ixz="0" iyy="0.01" iyz="0" izz="0.01" />
-      </inertial>
+      <xacro:default_inertial/>
       <visual>
         <origin xyz="0 0 0" rpy="0 0 0" />
@@ -226,15 +191,11 @@
       <child link="${name}_7_link"/>
       <axis xyz="0 0 1" />
-      <calibration rising="${arm_7_ref}"/>
-      <dynamics damping="5" />
-      <limit effort="9.6" velocity="2.0" lower="-6.25" upper="6.25" />
-      <safety_controller k_position="20" k_velocity="25" soft_lower_limit="${-6.25 + 0.01}" soft_upper_limit="${6.25 - 0.01}" />
+      <dynamics damping="5" />
+      <limit effort="9.6" velocity="2.0" lower="-3.1415" upper="3.1415" />
+      <!--limit effort="9.6" velocity="2.0" lower="-6.25" upper="6.25" /-->
+      <!--safety_controller k_position="20" k_velocity="25" soft_lower_limit="${-6.25 + 0.01}" soft_upper_limit="${6.25 - 0.01}" /-->
     </joint>
     <link name="${name}_7_link">
-      <inertial>
-        <origin xyz="0 0 0" rpy="0 0 0"/>
-        <mass value="1.120198"/>
-        <inertia ixx="0.01" ixy="0" ixz="0" iyy="0.01" iyz="0" izz="0.01" />
-      </inertial>
+      <xacro:default_inertial/>
       <visual>
         <origin xyz="0 0 0" rpy="0 0 0" />

File: schunk_description/urdf/lwa4d/lwa4d.urdf.xacro (robot description, xacro)
@@ -1,42 +1,54 @@
 <?xml version="1.0"?>
 <robot xmlns:xacro="http://www.ros.org/wiki/xacro">
+  <property name="safety_offset" value="0.02"/>
   <xacro:include filename="$(find schunk_description)/urdf/lwa4d/lwa4d.gazebo.xacro"/>
   <xacro:include filename="$(find schunk_description)/urdf/lwa4d/lwa4d.transmission.xacro"/>
-  <xacro:macro name="schunk_lwa4d" params="parent name *origin arm_1_ref arm_2_ref arm_3_ref arm_4_ref arm_5_ref arm_6_ref arm_7_ref">
-    <!-- joint between base_link and arm_base_link -->
-    <joint name="${name}_base_joint" type="fixed">
-      <insert_block name="origin"/>
-      <parent link="${parent}"/>
-      <child link="${name}_base_link"/>
-    </joint>
-     <link name="${name}_base_link">
-      <xacro:default_inertial/>
-<!--
-      <xacro:cylinder_inertial radius="0.045" length="0.03" mass="3.6">
-        <origin xyz="0 0 0.015" rpy="0 0 0"/>
-       </xacro:cylinder_inertial>
--->
-       <visual>
-        <origin xyz="0 0 0.015" rpy="0 0 0"/>
-         <geometry>
-          <cylinder radius="0.045" length="0.03"/>
-         </geometry>
-         <material name="Schunk/Black"/>
-       </visual>
-       <collision>
-        <origin xyz="0 0 0.015" rpy="0 0 0"/>
-         <geometry>
-          <cylinder radius="0.045" length="0.03"/>
-         </geometry>
-       </collision>
-    </link>
-    <!-- joint between arm_0_link and arm_1_link -->
+  <xacro:macro name="schunk_lwa4d" params="parent name *origin has_podest">
+    <xacro:if value="${has_podest}">
+      <!-- joint between base_link and lwa4p_extended_connector_link -->
+      <joint name="${name}_podest_joint" type="fixed">
+        <insert_block name="origin" />
+        <parent link="${parent}"/>
+        <child link="${name}_podest_link"/>
+      </joint>
+      <link name="${name}_podest_link">
+        <xacro:default_inertial/>
+        <visual>
+          <origin xyz="0 0 0" rpy="0 0 0" />
+          <geometry>
+            <cylinder radius="0.03" length="0.05"/>
+          </geometry>
+        </visual>
+        <collision>
+          <origin xyz="0 0 0" rpy="0 0 0" />
+          <geometry>
+            <cylinder radius="0.03" length="0.05"/>
+          </geometry>
+        </collision>
+      </link>
+      <joint name="${name}_base_joint" type="fixed">
+        <origin xyz="0 0 0.175" rpy="0 ${M_PI} 0" />
+        <parent link="${name}_podest_link"/>
+        <child link="${name}_base_link"/>
+      </joint>
+    </xacro:if>
+    <xacro:unless value="${has_podest}">
+      <!-- joint between base_link and lwa4p_extended_connector_link -->
+      <joint name="${name}_base_joint" type="fixed">
+        <insert_block name="origin" />
+        <parent link="${parent}"/>
+        <child link="${name}_base_link"/>
+      </joint>
+    </xacro:unless>
+    <link name="${name}_base_link">
+      <xacro:default_inertial/>
+    </link>
+    <!-- joint between arm_base_link and arm_1_link -->
     <joint name="${name}_1_joint" type="revolute">
-      <origin xyz="0 0 0.15" rpy="0 -${M_PI} 0"/>
+      <origin xyz="0 0 0" rpy="0 0 0" />
       <parent link="${name}_base_link"/>
       <child link="${name}_1_link"/>
       <axis xyz="0 0 1"/>
-      <calibration rising="${arm_1_ref}"/>
-      <limit effort="216" velocity="0.43633" lower="-${M_PI}" upper="${M_PI}"/>
+      <limit effort="216" velocity="0.43633" lower="${-M_PI+safety_offset}" upper="${M_PI-safety_offset}"/>
     </joint>
     <link name="${name}_1_link">
@@ -67,6 +79,5 @@
       <child link="${name}_2_link"/>
       <axis xyz="0 0 1"/>
-      <calibration rising="${arm_2_ref}"/>
-      <limit effort="216" velocity="0.43633" lower="-${M_PI}" upper="${M_PI}"/>
+      <limit effort="216" velocity="0.43633" lower="${-2.14 + safety_offset}" upper="${2.14 - safety_offset}"/>
     </joint>
     <link name="${name}_2_link">
@@ -97,6 +108,5 @@
       <child link="${name}_3_link"/>
       <axis xyz="0 0 1"/>
-      <calibration rising="${arm_3_ref}"/>
-      <limit effort="81.5" velocity="0.4189" lower="-${M_PI}" upper="${M_PI}"/>
+      <limit effort="81.5" velocity="0.4189" lower="${-M_PI + safety_offset}" upper="${M_PI - safety_offset}"/>
     </joint>
     <link name="${name}_3_link">
@@ -127,6 +137,5 @@
       <child link="${name}_4_link"/>
       <axis xyz="0 0 1"/>
-      <calibration rising="${arm_4_ref}"/>
-      <limit effort="81.5" velocity="0.4189" lower="-${M_PI}" upper="${M_PI}"/>
+      <limit effort="81.5" velocity="0.4189" lower="${-2.18 + safety_offset}" upper="${2.18 - safety_offset}"/>
     </joint>
     <link name="${name}_4_link">
@@ -157,6 +166,5 @@
       <child link="${name}_5_link"/>
       <axis xyz="0 0 1"/>
-      <calibration rising="${arm_5_ref}"/>
-      <limit effort="20.7" velocity="0.43633" lower="-${M_PI}" upper="${M_PI}"/>
+      <limit effort="20.7" velocity="0.43633" lower="${-M_PI + safety_offset}" upper="${M_PI - safety_offset}"/>
     </joint>
     <link name="${name}_5_link">
@@ -187,6 +195,5 @@
       <child link="${name}_6_link"/>
       <axis xyz="0 0 1"/>
-      <calibration rising="${arm_6_ref}"/>
-      <limit effort="15" velocity="1.2566" lower="-2.0943951" upper="2.0943951"/>
+      <limit effort="15" velocity="1.2566" lower="${-2.09 + safety_offset}" upper="${2.09 - safety_offset}"/>
     </joint>
     <link name="${name}_6_link">
@@ -217,6 +224,5 @@
       <child link="${name}_7_link"/>
       <axis xyz="0 0 1"/>
-      <calibration rising="${arm_7_ref}"/>
-      <limit effort="15" velocity="1.2566" lower="-2.0943951" upper="2.0943951"/>
+      <limit effort="15" velocity="1.2566" lower="${-2.96 + safety_offset}" upper="${2.96 - safety_offset}"/>
     </joint>
     <link name="${name}_7_link">

File: schunk_description/urdf/lwa4p/lwa4p.urdf.xacro (robot description, xacro)
@@ -1,45 +1,55 @@
 <?xml version="1.0"?>
 <robot xmlns:xacro="http://www.ros.org/wiki/xacro">
+  <property name="safety_offset" value="0.02"/>
   <xacro:include filename="$(find schunk_description)/urdf/lwa4p/lwa4p.gazebo.xacro" />
   <xacro:include filename="$(find schunk_description)/urdf/lwa4p/lwa4p.transmission.xacro" />
-  <xacro:macro name="schunk_lwa4p" params="parent name *origin arm_1_ref arm_2_ref arm_3_ref arm_4_ref arm_5_ref arm_6_ref">
-    <!-- joint between base_link and arm_0_link -->
-    <joint name="${name}_0_joint" type="fixed">
-      <insert_block name="origin" />
-      <parent link="${parent}"/>
-      <child link="${name}_0_link"/>
-    </joint>
-    <link name="${name}_0_link">
-      <xacro:default_inertial/>
-<!--
-      <inertial>
-        <origin xyz="0 0 0" rpy="0 0 0" />
-        <mass value="0.29364"/>
-        <inertia ixx="0.01" ixy="0" ixz="0" iyy="0.01" iyz="0" izz="0.01" />
-      </inertial>
--->
-      <visual>
-        <origin xyz="0 0 0" rpy="0 0 0" />
-        <geometry>
-          <mesh filename="package://schunk_description/meshes/lwa4p/arm_0_link.stl" />
-        </geometry>
-        <material name="Schunk/LightGrey" />
-      </visual>
-      <collision>
-        <origin xyz="0 0 0" rpy="0 0 0" />
-        <geometry>
-          <mesh filename="package://schunk_description/meshes/lwa4p/arm_0_link.stl" />
-        </geometry>
-      </collision>
+  <xacro:macro name="schunk_lwa4p" params="parent name *origin has_podest">
+    <xacro:if value="${has_podest}">
+      <!-- joint between base_link and lwa4p_extended_connector_link -->
+      <joint name="${name}_podest_joint" type="fixed">
+        <insert_block name="origin" />
+        <parent link="${parent}"/>
+        <child link="${name}_podest_link"/>
+      </joint>
+      <link name="${name}_podest_link">
+        <xacro:default_inertial/>
+        <visual>
+          <origin xyz="0 0 0" rpy="0 ${M_PI} 0" />
+          <geometry>
+          <mesh filename="package://schunk_description/meshes/lwa4p/arm_base_link.stl" />
+          </geometry>
+        </visual>
+        <collision>
+          <origin xyz="0 0 0" rpy="0 ${M_PI} 0" />
+          <geometry>
+          <mesh filename="package://schunk_description/meshes/lwa4p/arm_base_link.stl" />
+          </geometry>
+        </collision>
+      </link>
+      <joint name="${name}_base_joint" type="fixed">
+        <origin xyz="0 0 0.10" rpy="0 0 0" />
+        <parent link="${name}_podest_link"/>
+        <child link="${name}_base_link"/>
+      </joint>
+    </xacro:if>
+    <xacro:unless value="${has_podest}">
+      <!-- joint between base_link and lwa4p_extended_connector_link -->
+      <joint name="${name}_base_joint" type="fixed">
+        <insert_block name="origin" />
+        <parent link="${parent}"/>
+        <child link="${name}_base_link"/>
+      </joint>
+    </xacro:unless>
+    <link name="${name}_base_link">
+      <xacro:default_inertial/>
     </link>
     <!-- joint between arm_0_link and arm_1_link -->
     <joint name="${name}_1_joint" type="revolute">
-      <origin xyz="0 0 0.11" rpy="0 0 0"/>
-      <parent link="${name}_0_link"/>
+      <origin xyz="0 0 0" rpy="0 0 0" />
+      <parent link="${name}_base_link"/>
       <child link="${name}_1_link"/>
       <axis xyz="0 0 1"/>
-      <calibration rising="${arm_1_ref}"/>
-      <limit effort="370" velocity="2.0" lower="-6.2831853" upper="6.2831853"/>
-      <!--safety_controller k_position="20" k_velocity="50" soft_lower_limit="${-6.2831853 + 0.01}" soft_upper_limit="${6.2831853 - 0.01}" /-->
+      <limit effort="370" velocity="2.0" lower="${-6.28 + safety_offset}" upper="${6.28 - safety_offset}"/>
+      <!--safety_controller k_position="20" k_velocity="50" soft_lower_limit="${-6.28 + 0.01}" soft_upper_limit="${6.28 - 0.01}" /-->
     </joint>
     <link name="${name}_1_link">
@@ -72,7 +82,6 @@
       <child link="${name}_2_link"/>
       <axis xyz="0 0 1"/>
-      <calibration rising="${arm_2_ref}"/>
-      <limit effort="370" velocity="2.0" lower="-2.0943951" upper="2.0943951"/>
-      <!--safety_controller k_position="20" k_velocity="50" soft_lower_limit="${-2.0943 + 0.01}" soft_upper_limit="${2.0943 - 0.01}" /-->
+      <limit effort="370" velocity="2.0" lower="${-2.09 + safety_offset}" upper="${2.09 - safety_offset}"/>
+      <!--safety_controller k_position="20" k_velocity="50" soft_lower_limit="${-2.09 + 0.01}" soft_upper_limit="${2.09 - 0.01}" /-->
     </joint>
     <link name="${name}_2_link">
@@ -105,7 +114,6 @@
       <child link="${name}_3_link"/>
       <axis xyz="0 0 1"/>
-      <calibration rising="${arm_3_ref}"/>
-      <limit effort="176" velocity="2.0" lower="-6.2831853" upper="6.2831853"/>
-      <!--safety_controller k_position="20" k_velocity="25" soft_lower_limit="${-6.2831853 + 0.01}" soft_upper_limit="${6.2831853 - 0.01}" /-->
+      <limit effort="176" velocity="2.0" lower="${-6.28 + safety_offset}" upper="${6.28 - safety_offset}"/>
+      <!--safety_controller k_position="20" k_velocity="25" soft_lower_limit="${-6.28 + 0.01}" soft_upper_limit="${6.28 - 0.01}" /-->
     </joint>
     <link name="${name}_3_link">
@@ -138,7 +146,6 @@
       <child link="${name}_4_link"/>
       <axis xyz="0 0 1" />
-      <calibration rising="${arm_4_ref}"/>
-      <limit effort="176" velocity="2.0" lower="-2.0943951" upper="2.0943951"/>
-      <!--safety_controller k_position="20" k_velocity="25" soft_lower_limit="${-2.0943951 + 0.01}" soft_upper_limit="${2.0943951 - 0.01}" /-->
+      <limit effort="176" velocity="2.0" lower="${-2.09 + safety_offset}" upper="${2.09 - safety_offset}"/>
+      <!--safety_controller k_position="20" k_velocity="25" soft_lower_limit="${-2.09 + 0.01}" soft_upper_limit="${2.09 - 0.01}" /-->
     </joint>
     <link name="${name}_4_link">
@@ -171,7 +178,6 @@
       <child link="${name}_5_link"/>
       <axis xyz="0 0 1" />
-      <calibration rising="${arm_5_ref}"/>
-      <limit effort="41.6" velocity="2.0" lower="-6.2831853" upper="6.2831853" />
-      <!--safety_controller k_position="20" k_velocity="25" soft_lower_limit="${-6.2831853 + 0.01}" soft_upper_limit="${6.2831853 - 0.01}" /-->
+      <limit effort="41.6" velocity="2.0" lower="${-6.28 + safety_offset}" upper="${6.28 - safety_offset}" />
+      <!--safety_controller k_position="20" k_velocity="25" soft_lower_limit="${-6.28 + 0.01}" soft_upper_limit="${6.28 - 0.01}" /-->
     </joint>
     <link name="${name}_5_link">
@@ -204,7 +210,6 @@
       <child link="${name}_6_link"/>
       <axis xyz="0 0 1" />
-      <calibration rising="${arm_6_ref}"/>
-      <limit effort="20.1" velocity="2.0" lower="-2.0943951" upper="2.0943951" />
-      <!--safety_controller k_position="20" k_velocity="25" soft_lower_limit="${-2.0943951 + 0.01}" soft_upper_limit="${2.0943951 - 0.01}" /-->
+      <limit effort="20.1" velocity="2.0" lower="${-2.09 + safety_offset}" upper="${2.09 - safety_offset}" />
+      <!--safety_controller k_position="20" k_velocity="25" soft_lower_limit="${-2.09 + 0.01}" soft_upper_limit="${2.09 - 0.01}" /-->
     </joint>
     <link name="${name}_6_link">
