Commit message: Imported upstream version '0.6.3' of 'upstream'

File: schunk_description/urdf/lwa4p_extended/lwa4p_extended.urdf.xacro (robot description, xacro)
@@ -1,21 +1,52 @@
 <?xml version="1.0"?>
 <robot xmlns:xacro="http://www.ros.org/wiki/xacro">
+  <property name="safety_offset" value="0.02"/>
   <xacro:include filename="$(find schunk_description)/urdf/lwa4p_extended/lwa4p_extended.gazebo.xacro" />
   <xacro:include filename="$(find schunk_description)/urdf/lwa4p_extended/lwa4p_extended.transmission.xacro" />
-  <xacro:macro name="schunk_lwa4p_extended" params="parent name *origin arm_1_ref arm_2_ref arm_3_ref arm_4_ref arm_5_ref arm_6_ref arm_7_ref">
-    <!-- joint between base_link and lwa4p_extended_connector_link -->
-    <joint name="${name}_base_joint" type="fixed">
-      <insert_block name="origin" />
-      <parent link="${parent}"/>
-      <child link="${name}_base_link"/>
-    </joint>
+  <xacro:macro name="schunk_lwa4p_extended" params="parent name *origin has_podest">
+    <xacro:if value="${has_podest}">
+      <!-- joint between base_link and lwa4p_extended_connector_link -->
+      <joint name="${name}_podest_joint" type="fixed">
+        <insert_block name="origin" />
+        <parent link="${parent}"/>
+        <child link="${name}_podest_link"/>
+      </joint>
+      <link name="${name}_podest_link">
+        <xacro:default_inertial/>
+        <visual>
+          <origin xyz="0 0 0" rpy="0 0 0" />
+          <geometry>
+            <cylinder radius="0.03" length="0.05"/>
+          </geometry>
+        </visual>
+        <collision>
+          <origin xyz="0 0 0" rpy="0 0 0" />
+          <geometry>
+            <cylinder radius="0.03" length="0.05"/>
+          </geometry>
+        </collision>
+      </link>
+      <joint name="${name}_base_joint" type="fixed">
+        <origin xyz="0 0 0.025" rpy="0 0 0" />
+        <parent link="${name}_podest_link"/>
+        <child link="${name}_base_link"/>
+      </joint>
+    </xacro:if>
+    <xacro:unless value="${has_podest}">
+      <!-- joint between base_link and lwa4p_extended_connector_link -->
+      <joint name="${name}_base_joint" type="fixed">
+        <insert_block name="origin" />
+        <parent link="${parent}"/>
+        <child link="${name}_base_link"/>
+      </joint>
+    </xacro:unless>
     <!-- static part of PRL100 -->
     <link name="${name}_base_link">
       <xacro:default_inertial/>
-<!--
+  <!--
       <xacro:cylinder_inertial radius="0.056" length="0.12" mass="2.0">
         <origin xyz="0 0 ${0.12/2}" rpy="0 0 0" />
       </xacro:cylinder_inertial>
--->
+  -->
       <visual>
         <origin xyz="0 0 0" rpy="0 0 0" />
@@ -33,11 +64,10 @@
     <!-- joint between arm_base_link and arm_1_link -->
     <joint name="${name}_1_joint" type="revolute">
-      <origin xyz="0 0 ${0.134+0.005}" rpy="0 0 0" />
-      <parent link="${name}_base_link" />
+      <origin xyz="0 0 0.139" rpy="0 0 0" />
+      <parent link="${name}_base_link"/>
       <child link="${name}_1_link" />
       <axis xyz="0 0 1"/>
-      <calibration rising="${arm_1_ref}"/>
-      <dynamics damping="0" friction="0"/>
-      <limit effort="81.5" velocity="0.42" lower="-4.712" upper="4.712"/>   <!--Theoricarl limit +/-270 , Real Limit +/- 270-->
+      <dynamics damping="0" friction="0"/>
+      <limit effort="81.5" velocity="0.66" lower="${-4.71 + safety_offset}" upper="${4.71 - safety_offset}"/>   <!--Theoretical limit +/-270 , Real Limit +/- 270-->
       <!--safety_controller k_position="20" k_velocity="50" soft_lower_limit="${-M_PI + 0.01}" soft_upper_limit="${M_PI - 0.01}" /-->
     </joint>
@@ -71,7 +101,6 @@
       <child link="${name}_2_link"/>
       <axis xyz="0 0 1"/>
-      <calibration rising="${arm_2_ref}"/>
-      <dynamics damping="0" friction="0"/>
-      <limit effort="48" velocity="1.2566" lower="-1.92" upper="1.92"/>   <!--Theoricarl limit +/-170 , Real Limit +/- 110 (self collision)-->
+      <dynamics damping="0" friction="0"/>
+      <limit effort="48" velocity="1.57" lower="${-1.91 + safety_offset}" upper="${1.91 - safety_offset}"/>   <!--Theoretical limit +/-170 , Real Limit +/- 110 (self collision)-->
       <!--safety_controller k_position="20" k_velocity="50" soft_lower_limit="${-2.0943 + 0.01}" soft_upper_limit="${2.0943 - 0.01}" /-->
     </joint>
@@ -104,7 +133,6 @@
       <child link="${name}_3_link"/>
       <axis xyz="0 0 1"/>
-      <calibration rising="${arm_3_ref}"/>
-      <dynamics damping="0" friction="0"/>
-      <limit effort="48" velocity="1.2566" lower="-2.967" upper="2.967"/>   <!--Theoricarl limit +/-170 , Real Limit +/- 170-->
+      <dynamics damping="0" friction="0"/>
+      <limit effort="48" velocity="1.57" lower="${-2.96 + safety_offset}" upper="${2.96 - safety_offset}"/>   <!--Theoretical limit +/-170 , Real Limit +/- 170-->
       <!--safety_controller k_position="20" k_velocity="25" soft_lower_limit="${-M_PI + 0.01}" soft_upper_limit="${M_PI - 0.01}" /-->
     </joint>
@@ -137,7 +165,6 @@
       <child link="${name}_4_link"/>
       <axis xyz="0 0 1" />
-      <calibration rising="${arm_4_ref}"/>
-      <dynamics damping="0" friction="0"/>
-      <limit effort="48" velocity="1.2566" lower="-2.618" upper="2.618"/>   <!--Theoricarl limit +/-170 , Real Limit +/- 150 (self collision)-->
+      <dynamics damping="0" friction="0"/>
+      <limit effort="48" velocity="1.57" lower="${-2.61 + safety_offset}" upper="${2.61 - safety_offset}"/>   <!--Theoretical limit +/-170 , Real Limit +/- 150 (self collision)-->
       <!--safety_controller k_position="20" k_velocity="25" soft_lower_limit="${-2.0943951 + 0.01}" soft_upper_limit="${2.0943951 - 0.01}" /-->
     </joint>
@@ -170,7 +197,6 @@
       <child link="${name}_5_link"/>
       <axis xyz="0 0 1" />
-      <calibration rising="${arm_5_ref}"/>
-      <dynamics damping="0" friction="0"/>
-      <limit effort="48" velocity="1.2566" lower="-2.967" upper="2.967"/>   <!--Theoricarl limit +/-170 , Real Limit +/- 170-->
+      <dynamics damping="0" friction="0"/>
+      <limit effort="48" velocity="1.57" lower="${-2.96 + safety_offset}" upper="${2.96 - safety_offset}"/>   <!--Theoretical limit +/-170 , Real Limit +/- 170-->
       <!--safety_controller k_position="20" k_velocity="25" soft_lower_limit="${-M_PI + 0.01}" soft_upper_limit="${M_PI - 0.01}" /-->
     </joint>
@@ -203,7 +229,6 @@
       <child link="${name}_6_link"/>
       <axis xyz="0 0 1" />
-      <calibration rising="${arm_6_ref}"/>
-      <dynamics damping="0" friction="0"/>
-      <limit effort="15" velocity="1.2566" lower="-2.443" upper="2.967"/>   <!--Theoricarl limit +/-170 , Real Limit -140/+170 (self collision)-->
+      <dynamics damping="0" friction="0"/>
+      <limit effort="15" velocity="2.09" lower="${-2.96 + safety_offset}" upper="${2.96 - safety_offset}"/>   <!--Theoretical limit +/-170 , Real Limit -140/+170 (self collision)-->
       <!--safety_controller k_position="20" k_velocity="25" soft_lower_limit="${-2.0943951 + 0.01}" soft_upper_limit="${2.0943951 - 0.01}" /-->
     </joint>
@@ -236,7 +261,6 @@
       <child link="${name}_7_link"/>
       <axis xyz="0 0 1" />
-      <calibration rising="${arm_7_ref}"/>
-      <dynamics damping="0" friction="0"/>
-      <limit effort="15" velocity="1.2566" lower="-2.967" upper="2.967"/>   <!--Theoricarl limit +/-170 , Real Limit +/- 170-->
+      <dynamics damping="0" friction="0"/>
+      <limit effort="15" velocity="2.09" lower="${-3.75 + safety_offset}" upper="${2.18 - safety_offset}"/>   <!--Theoretical limit +127/-215 , Real Limit +127/-215-->
       <!--safety_controller k_position="20" k_velocity="25" soft_lower_limit="${-2.0943951 + 0.01}" soft_upper_limit="${2.0943951 - 0.01}" /-->
     </joint>

File: schunk_description/urdf/pg70/pg70.urdf.xacro (robot description, xacro)
@@ -3,5 +3,5 @@
   <xacro:include filename="$(find schunk_description)/urdf/pg70/pg70.gazebo.xacro" />
   <xacro:include filename="$(find schunk_description)/urdf/pg70/pg70.transmission.xacro" />
-  <xacro:macro name="schunk_pg70" params="parent name *origin pg70_finger_left_ref pg70_finger_right_ref">
+  <xacro:macro name="schunk_pg70" params="parent name *origin">
     <joint name="${name}_palm_joint" type="fixed" >
       <parent link="${parent}" />
@@ -35,7 +35,6 @@
       <parent link="${name}_palm_link" />
       <child link="${name}_finger_left_link" />
-      <limit effort="100" lower="-0.001" upper="0.0345" velocity="2.0"/>
-      <calibration rising="${pg70_finger_left_ref}"/>
-      <origin xyz="0 0.0105 0.0789" rpy="0 0 0"/>
+      <limit effort="100" lower="-0.001" upper="0.061" velocity="2.0"/>
+      <origin xyz="0 0 0.0789" rpy="0 0 0"/>
       <axis xyz="0 1 0" />
     </joint>
@@ -67,7 +66,6 @@
       <parent link="${name}_palm_link" />
       <child link="${name}_finger_right_link" />
-      <limit effort="100" lower="-0.001" upper="0.0345" velocity="2.0"/>
-      <calibration rising="${pg70_finger_right_ref}"/>
-      <origin xyz="0 -0.0105 0.0789" rpy="-0 0 0"/>
+      <limit effort="100" lower="-0.001" upper="0.061" velocity="2.0"/>
+      <origin xyz="0 0 0.0789" rpy="-0 0 0"/>
       <axis xyz="0 -1 0" />
     </joint>
