Commit message: Rebase from 'upstream'

File: schunk_description/urdf/lwa4d/lwa4d.urdf.xacro (robot description, xacro)
@@ -4,5 +4,17 @@
   <xacro:include filename="$(find schunk_description)/urdf/lwa4d/lwa4d.gazebo.xacro"/>
   <xacro:include filename="$(find schunk_description)/urdf/lwa4d/lwa4d.transmission.xacro"/>
-  <xacro:macro name="schunk_lwa4d" params="parent name *origin has_podest">
+  <xacro:macro name="axis_config" params="invert">
+    <xacro:if value="${invert}">
+      <axis xyz="0 0 1" />
+    </xacro:if>
+    <xacro:unless value="${invert}">
+      <axis xyz="0 0 -1" />
+    </xacro:unless>
+  </xacro:macro>
+  <!-- invert_* is a xacro parameter to be used to adapt the urdf according to your hardware setup.
+       use invert_*:=true if  motors are inverted in the firmware.
+       use invert_*:=false if motors are not inverted in the firmware.
+  -->
+  <xacro:macro name="schunk_lwa4d_custom" params="parent name *origin has_podest invert_j1 invert_j2 invert_j3 invert_j4 invert_j5 invert_j6 invert_j7">
     <xacro:if value="${has_podest}">
       <!-- joint between base_link and lwa4p_extended_connector_link -->
@@ -15,18 +27,17 @@
         <xacro:default_inertial/>
         <visual>
-          <origin xyz="0 0 0" rpy="0 0 0" />
           <geometry>
-            <cylinder radius="0.03" length="0.05"/>
+            <mesh filename="package://schunk_description/meshes/lwa4d/arm_podest_link.stl"/>
           </geometry>
+          <material name="Schunk/LightGrey"/>
         </visual>
         <collision>
-          <origin xyz="0 0 0" rpy="0 0 0" />
           <geometry>
-            <cylinder radius="0.03" length="0.05"/>
+            <mesh filename="package://schunk_description/meshes/lwa4d/arm_podest_link.stl"/>
           </geometry>
         </collision>
       </link>
       <joint name="${name}_base_joint" type="fixed">
-        <origin xyz="0 0 0.175" rpy="0 ${M_PI} 0" />
+        <origin xyz="0 0 0.140" rpy="0 0 0" />
         <parent link="${name}_podest_link"/>
         <child link="${name}_base_link"/>
@@ -49,5 +60,5 @@
       <parent link="${name}_base_link"/>
       <child link="${name}_1_link"/>
-      <axis xyz="0 0 1"/>
+      <xacro:axis_config invert="${invert_j1}"/>
       <limit effort="216" velocity="0.43633" lower="${-M_PI+safety_offset}" upper="${M_PI-safety_offset}"/>
     </joint>
@@ -60,5 +71,4 @@
 -->
       <visual>
-        <origin xyz="0 0 -0.15" rpy="0 0 ${M_PI}"/>
         <geometry>
           <mesh filename="package://schunk_description/meshes/lwa4d/arm_1_link.stl"/>
@@ -67,5 +77,4 @@
       </visual>
       <collision>
-        <origin xyz="0 0 -0.15" rpy="0 0 ${M_PI}"/>
         <geometry>
           <mesh filename="package://schunk_description/meshes/lwa4d/arm_1_link.stl"/>
@@ -75,8 +84,8 @@
     <!-- joint between arm_1_link and arm_2_link -->
     <joint name="${name}_2_joint" type="revolute">
-      <origin xyz="0 0 -0.15" rpy="-${M_PI/2} 0 0"/>
+      <origin xyz="0 0 0.240" rpy="-${M_PI/2} -${M_PI/2} 0"/>
       <parent link="${name}_1_link"/>
       <child link="${name}_2_link"/>
-      <axis xyz="0 0 1"/>
+      <xacro:axis_config invert="${invert_j2}"/>
       <limit effort="216" velocity="0.43633" lower="${-2.14 + safety_offset}" upper="${2.14 - safety_offset}"/>
     </joint>
@@ -89,5 +98,4 @@
 -->
       <visual>
-        <origin xyz="0 0 0" rpy="0 0 ${M_PI}"/>
         <geometry>
           <mesh filename="package://schunk_description/meshes/lwa4d/arm_2_link.stl"/>
@@ -96,5 +104,4 @@
       </visual>
       <collision>
-        <origin xyz="0 0 0" rpy="0 0 ${M_PI}"/>
         <geometry>
           <mesh filename="package://schunk_description/meshes/lwa4d/arm_2_link_collision.stl"/>
@@ -104,8 +111,8 @@
     <!-- joint between arm_2_link and arm_3_link -->
     <joint name="${name}_3_joint" type="revolute">
-      <origin xyz="0 0 0" rpy="${M_PI/2} 0 0"/>
+      <origin xyz="0 0 0" rpy="${M_PI/2} 0 ${M_PI/2}"/>
       <parent link="${name}_2_link"/>
       <child link="${name}_3_link"/>
-      <axis xyz="0 0 1"/>
+      <xacro:axis_config invert="${invert_j3}"/>
       <limit effort="81.5" velocity="0.4189" lower="${-M_PI + safety_offset}" upper="${M_PI - safety_offset}"/>
     </joint>
@@ -118,5 +125,4 @@
 -->
       <visual>
-        <origin xyz="0 0 -0.39" rpy="0 0 ${M_PI}"/>
         <geometry>
           <mesh filename="package://schunk_description/meshes/lwa4d/arm_3_link.stl"/>
@@ -125,5 +131,4 @@
       </visual>
       <collision>
-        <origin xyz="0 0 -0.39" rpy="0 0 ${M_PI}"/>
         <geometry>
           <mesh filename="package://schunk_description/meshes/lwa4d/arm_3_link_collision.stl"/>
@@ -133,8 +138,8 @@
     <!-- joint between arm_3_link and arm_4_link -->
     <joint name="${name}_4_joint" type="revolute">
-      <origin xyz="0 0 -0.39" rpy="-${M_PI/2} 0 0"/>
+      <origin xyz="0 0 0.328" rpy="-${M_PI/2} -${M_PI/2} 0"/>
       <parent link="${name}_3_link"/>
       <child link="${name}_4_link"/>
-      <axis xyz="0 0 1"/>
+      <xacro:axis_config invert="${invert_j4}"/>
       <limit effort="81.5" velocity="0.4189" lower="${-2.18 + safety_offset}" upper="${2.18 - safety_offset}"/>
     </joint>
@@ -147,5 +152,4 @@
 -->
       <visual>
-        <origin xyz="0 0 0" rpy="0 0 ${M_PI}"/>
         <geometry>
           <mesh filename="package://schunk_description/meshes/lwa4d/arm_4_link.stl"/>
@@ -154,5 +158,4 @@
       </visual>
       <collision>
-        <origin xyz="0 0 0" rpy="0 0 ${M_PI}"/>
         <geometry>
           <mesh filename="package://schunk_description/meshes/lwa4d/arm_4_link_collision.stl"/>
@@ -162,8 +165,8 @@
     <!-- joint between arm_4_link and arm_5_link -->
     <joint name="${name}_5_joint" type="revolute">
-      <origin xyz="0 0 0" rpy="${M_PI/2} 0 0"/>
+      <origin xyz="0 0 0" rpy="${M_PI/2} 0 ${M_PI/2}"/>
       <parent link="${name}_4_link"/>
       <child link="${name}_5_link"/>
-      <axis xyz="0 0 1"/>
+      <xacro:axis_config invert="${invert_j5}"/>
       <limit effort="20.7" velocity="0.43633" lower="${-M_PI + safety_offset}" upper="${M_PI - safety_offset}"/>
     </joint>
@@ -176,5 +179,4 @@
 -->
       <visual>
-        <origin xyz="0 0 -0.323" rpy="0 0 ${M_PI}"/>
         <geometry>
           <mesh filename="package://schunk_description/meshes/lwa4d/arm_5_link.stl"/>
@@ -183,5 +185,4 @@
       </visual>
       <collision>
-        <origin xyz="0 0 -0.323" rpy="0 0 ${M_PI}"/>
         <geometry>
           <mesh filename="package://schunk_description/meshes/lwa4d/arm_5_link_collision.stl"/>
@@ -191,8 +192,8 @@
     <!-- joint between arm_5_link and arm_6_link -->
     <joint name="${name}_6_joint" type="revolute">
-      <origin xyz="0 0 -0.323" rpy="-${M_PI/2} 0 0"/>
+      <origin xyz="0 0 0.323" rpy="-${M_PI/2} -${M_PI/2} 0"/>
       <parent link="${name}_5_link"/>
       <child link="${name}_6_link"/>
-      <axis xyz="0 0 1"/>
+      <xacro:axis_config invert="${invert_j6}"/>
       <limit effort="15" velocity="1.2566" lower="${-2.09 + safety_offset}" upper="${2.09 - safety_offset}"/>
     </joint>
@@ -205,5 +206,4 @@
 -->
       <visual>
-        <origin xyz="0 0 0" rpy="0 ${M_PI} 0"/>
         <geometry>
           <mesh filename="package://schunk_description/meshes/lwa4d/arm_6_link.stl"/>
@@ -212,5 +212,4 @@
       </visual>
       <collision>
-        <origin xyz="0 0 0" rpy="0 ${M_PI} 0"/>
         <geometry>
           <mesh filename="package://schunk_description/meshes/lwa4d/arm_6_link_collision.stl"/>
@@ -220,8 +219,8 @@
     <!-- joint between arm_6_link and arm_7_link -->
     <joint name="${name}_7_joint" type="revolute">
-      <origin xyz="0 0 0" rpy="-${M_PI/2} 0 0"/>
+      <origin xyz="0 0 0" rpy="${M_PI/2} 0 ${M_PI/2}"/>
       <parent link="${name}_6_link"/>
       <child link="${name}_7_link"/>
-      <axis xyz="0 0 1"/>
+      <xacro:axis_config invert="${invert_j7}"/>
       <limit effort="15" velocity="1.2566" lower="${-2.96 + safety_offset}" upper="${2.96 - safety_offset}"/>
     </joint>
@@ -234,16 +233,22 @@
 -->
       <visual>
-        <origin xyz="0 0 0.06" rpy="0 0 0"/>
-        <geometry>
-          <cylinder radius="0.03" length="0.035"/>
-        </geometry>
-        <material name="Schunk/LightGrey"/>
-      </visual>
-      <collision>
-        <origin xyz="0 0 0.06" rpy="0 0 0"/>
-        <geometry>
-          <cylinder radius="0.03" length="0.035"/>
-        </geometry>
-      </collision>
+        <geometry>
+          <mesh filename="package://schunk_description/meshes/lwa4d/arm_7_link.stl"/>
+        </geometry>
+        <material name="Schunk/LightGrey"/>
+      </visual>
+      <collision>
+        <geometry>
+          <mesh filename="package://schunk_description/meshes/lwa4d/arm_7_link.stl"/>
+        </geometry>
+      </collision>
+    </link>
+    <joint name="${name}_ee_joint" type="fixed">
+      <origin xyz="0 0 0.0824" rpy="0 0 0"/>
+      <parent link="${name}_7_link"/>
+      <child link="${name}_ee_link"/>
+    </joint>
+    <link name="${name}_ee_link">
+      <xacro:default_inertial/>
     </link>
     <!-- extensions -->
@@ -251,3 +256,20 @@
     <xacro:schunk_lwa4d_transmission name="${name}"/>
   </xacro:macro>
+  <!-- use_factory_setings is a xacro parameter to be used to adapt the urdf according to your hardware setup.
+       use_factory_settings:=true if you have not modified the schunk firmware.
+       use_factory_settings:=false if you have modified the schunk firmware to follow DH parameters (you have inverted the PRL+ motors j1-j5)
+       if you are using custom firmware settings, use schunk_lwa4d_custom
+  -->
+  <xacro:macro name="schunk_lwa4d" params="parent name *origin has_podest use_factory_settings:=false">
+    <xacro:if value="${use_factory_settings}">
+      <xacro:schunk_lwa4d_custom parent="${parent}" name="${name}" has_podest="${has_podest}" invert_j1="false" invert_j2="false" invert_j3="false" invert_j4="false" invert_j5="false" invert_j6="true" invert_j7="true">
+        <xacro:insert_block name="origin" />
+      </xacro:schunk_lwa4d_custom>
+    </xacro:if>
+    <xacro:unless value="${use_factory_settings}">
+      <xacro:schunk_lwa4d_custom parent="${parent}" name="${name}" has_podest="${has_podest}" invert_j1="true" invert_j2="true" invert_j3="true" invert_j4="true" invert_j5="true" invert_j6="true" invert_j7="true">
+        <xacro:insert_block name="origin" />
+      </xacro:schunk_lwa4d_custom>
+    </xacro:unless>
+  </xacro:macro>
 </robot>

File: schunk_description/urdf/lwa4p/lwa4p.urdf.xacro (robot description, xacro)
@@ -50,5 +50,5 @@
       <child link="${name}_1_link"/>
       <axis xyz="0 0 1"/>
-      <limit effort="370" velocity="2.0" lower="${-6.28 + safety_offset}" upper="${6.28 - safety_offset}"/>
+      <limit effort="370" velocity="1.26" lower="${-2.967 + safety_offset}" upper="${2.967 - safety_offset}"/>
       <!--safety_controller k_position="20" k_velocity="50" soft_lower_limit="${-6.28 + 0.01}" soft_upper_limit="${6.28 - 0.01}" /-->
     </joint>
@@ -82,5 +82,5 @@
       <child link="${name}_2_link"/>
       <axis xyz="0 0 1"/>
-      <limit effort="370" velocity="2.0" lower="${-2.09 + safety_offset}" upper="${2.09 - safety_offset}"/>
+      <limit effort="370" velocity="1.26" lower="${-2.967 + safety_offset}" upper="${2.967 - safety_offset}"/>
       <!--safety_controller k_position="20" k_velocity="50" soft_lower_limit="${-2.09 + 0.01}" soft_upper_limit="${2.09 - 0.01}" /-->
     </joint>
@@ -114,5 +114,5 @@
       <child link="${name}_3_link"/>
       <axis xyz="0 0 1"/>
-      <limit effort="176" velocity="2.0" lower="${-6.28 + safety_offset}" upper="${6.28 - safety_offset}"/>
+      <limit effort="176" velocity="1.26" lower="${-2.714 + safety_offset}" upper="${2.714 - safety_offset}"/>
       <!--safety_controller k_position="20" k_velocity="25" soft_lower_limit="${-6.28 + 0.01}" soft_upper_limit="${6.28 - 0.01}" /-->
     </joint>
@@ -146,5 +146,5 @@
       <child link="${name}_4_link"/>
       <axis xyz="0 0 1" />
-      <limit effort="176" velocity="2.0" lower="${-2.09 + safety_offset}" upper="${2.09 - safety_offset}"/>
+      <limit effort="176" velocity="1.26" lower="${-2.967 + safety_offset}" upper="${2.967 - safety_offset}"/>
       <!--safety_controller k_position="20" k_velocity="25" soft_lower_limit="${-2.09 + 0.01}" soft_upper_limit="${2.09 - 0.01}" /-->
     </joint>
@@ -178,5 +178,5 @@
       <child link="${name}_5_link"/>
       <axis xyz="0 0 1" />
-      <limit effort="41.6" velocity="2.0" lower="${-6.28 + safety_offset}" upper="${6.28 - safety_offset}" />
+      <limit effort="41.6" velocity="1.26" lower="${-2.967 + safety_offset}" upper="${2.967 - safety_offset}" />
       <!--safety_controller k_position="20" k_velocity="25" soft_lower_limit="${-6.28 + 0.01}" soft_upper_limit="${6.28 - 0.01}" /-->
     </joint>
@@ -210,5 +210,5 @@
       <child link="${name}_6_link"/>
       <axis xyz="0 0 1" />
-      <limit effort="20.1" velocity="2.0" lower="${-2.09 + safety_offset}" upper="${2.09 - safety_offset}" />
+      <limit effort="20.1" velocity="1.26" lower="${-2.967 + safety_offset}" upper="${2.967 - safety_offset}" />
       <!--safety_controller k_position="20" k_velocity="25" soft_lower_limit="${-2.09 + 0.01}" soft_upper_limit="${2.09 - 0.01}" /-->
     </joint>

File: schunk_description/urdf/lwa4p_extended/lwa4p_extended.urdf.xacro (robot description, xacro)
@@ -97,5 +97,5 @@
     <!-- joint between arm_1_link and arm_2_link -->
     <joint name="${name}_2_joint" type="revolute">
-      <origin xyz="0 0 0.0915" rpy="1.5708 0 0"/>
+      <origin xyz="0 0 0.0915" rpy="${M_PI/2} 0 0"/>
       <parent link="${name}_1_link"/>
       <child link="${name}_2_link"/>
@@ -129,5 +129,5 @@
     <!-- joint between arm_2_link and arm_3_link -->
     <joint name="${name}_3_joint" type="revolute">
-      <origin xyz="0 0 0" rpy="-1.5708 0 0"/>
+      <origin xyz="0 0 0" rpy="-${M_PI/2} 0 0"/>
       <parent link="${name}_2_link"/>
       <child link="${name}_3_link"/>
@@ -161,5 +161,5 @@
     <!-- joint between arm_3_link and arm_4_link -->
     <joint name="${name}_4_joint" type="revolute">
-      <origin xyz="0 0 0.45360" rpy="1.5708 0 0" />
+      <origin xyz="0 0 0.45360" rpy="${M_PI/2} 0 0" />
       <parent link="${name}_3_link"/>
       <child link="${name}_4_link"/>
@@ -193,5 +193,5 @@
     <!-- joint between arm_4_link and arm_5_link -->
     <joint name="${name}_5_joint" type="revolute">
-      <origin xyz="0 0 0" rpy="-1.5708 0 0" />
+      <origin xyz="0 0 0" rpy="-${M_PI/2} 0 0" />
       <parent link="${name}_4_link"/>
       <child link="${name}_5_link"/>
@@ -225,5 +225,5 @@
     <!-- joint between arm_5_link and arm_6_link -->
     <joint name="${name}_6_joint" type="revolute">
-      <origin xyz="0 0 0.2986" rpy="1.5708 0 0" />
+      <origin xyz="0 0 0.2986" rpy="${M_PI/2} 0 0" />
       <parent link="${name}_5_link"/>
       <child link="${name}_6_link"/>
@@ -257,5 +257,5 @@
     <!-- joint between arm_6_link and arm_7_link -->
     <joint name="${name}_7_joint" type="revolute">
-      <origin xyz="0 0 0" rpy="-1.5708 0 0" />
+      <origin xyz="0 0 0" rpy="-${M_PI/2} 0 0" />
       <parent link="${name}_6_link"/>
       <child link="${name}_7_link"/>
