Commit message: Imported upstream version '0.6.14' of 'upstream'

File: schunk_description/urdf/common.xacro (robot description, xacro)
@@ -41,6 +41,6 @@
       <type>transmission_interface/SimpleTransmission</type>
       <joint name="${jname}_joint">
-        <hardwareInterface>PositionJointInterface</hardwareInterface>
-        <hardwareInterface>VelocityJointInterface</hardwareInterface>
+        <hardwareInterface>hardware_interface/PositionJointInterface</hardwareInterface>
+        <hardwareInterface>hardware_interface/VelocityJointInterface</hardwareInterface>
         <!--hardwareInterface>EffortJointInterface</hardwareInterface-->
       </joint>

File: schunk_description/urdf/pg70/pg70.urdf.xacro (robot description, xacro)
@@ -58,5 +58,5 @@
     </link>
     <joint name="${name}_finger_left_joint" type="prismatic" >
-      <origin xyz="0 0 0.0789" rpy="0 0 0"/>
+      <origin xyz="0 0.0055 0.0789" rpy="0 0 0"/>
       <parent link="${name}_palm_link" />
       <child link="${name}_finger_left_link" />
@@ -88,5 +88,5 @@
     </link>
     <joint name="${name}_finger_right_joint" type="prismatic" >
-      <origin xyz="0 0 0.0789" rpy="-0 0 0"/>
+      <origin xyz="0 -0.0055 0.0789" rpy="-0 0 0"/>
       <parent link="${name}_palm_link" />
       <child link="${name}_finger_right_link" />
